File: IN-8/Socket.kicad_pcb (KiCad board)
At the start: 2 copper layers, 220 x 65 mm, 19 parts, among them J1 CONNECTOR, J2 CONNECTOR, J3 CONNECTOR, J4 CONNECTOR, J5 CONNECTOR, J6 CONNECTOR, T1 TUBE, T2 TUBE, T3 TUBE, T4 TUBE, T5 TUBE, T6 TUBE

Commit message: Migrate to KiCAD 6
Other:
- net class Default removed
