File: Spacer/Spacer.kicad_pcb (KiCad board)
At the start: 2 copper layers, 65 x 10 mm, 0 parts

Commit message: Migrate to KiCAD 6
Other:
- net class Default removed
Changed lines of the file:
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@@
-(kicad_pcb (version 20171130) (host pcbnew "(5.1.10)-1")
+(kicad_pcb (version 20211014) (generator pcbnew)
   (general
     (thickness 1.6)
-    (drawings 14)
-    (tracks 0)
-    (zones 0)
-    (modules 0)
-    (nets 1)
   )
-  (page A4)
+  (paper "A4")
   (layers
-    (0 F.Cu signal)
-    (31 B.Cu signal)
-    (32 B.Adhes user)
-    (33 F.Adhes user)
-    (34 B.Paste user)
-    (35 F.Paste user)
-    (36 B.SilkS user)
-    (37 F.SilkS user)
-    (38 B.Mask user)
-    (39 F.Mask user)
-    (40 Dwgs.User user)
-    (41 Cmts.User user)
-    (42 Eco1.User user)
-    (43 Eco2.User user)
-    (44 Edge.Cuts user)
-    (45 Margin user)
-    (46 B.CrtYd user)
-    (47 F.CrtYd user)
-    (48 B.Fab user)
-    (49 F.Fab user)
+    (0 "F.Cu" signal)
+    (31 "B.Cu" signal)
+    (32 "B.Adhes" user "B.Adhesive")
+    (33 "F.Adhes" user "F.Adhesive")
+    (34 "B.Paste" user)
+    (35 "F.Paste" user)
+    (36 "B.SilkS" user "B.Silkscreen")
+    (37 "F.SilkS" user "F.Silkscreen")
+    (38 "B.Mask" user)
+    (39 "F.Mask" user)
+    (40 "Dwgs.User" user "User.Drawings")
+    (41 "Cmts.User" user "User.Comments")
+    (42 "Eco1.User" user "User.Eco1")
+    (43 "Eco2.User" user "User.Eco2")
+    (44 "Edge.Cuts" user)
+    (45 "Margin" user)
+    (46 "B.CrtYd" user "B.Courtyard")
+    (47 "F.CrtYd" user "F.Courtyard")
+    (48 "B.Fab" user)
+    (49 "F.Fab" user)
   )
   (setup
-    (last_trace_width 0.25)
-    (trace_clearance 0.2)
-    (zone_clearance 0.508)
-    (zone_45_only no)
-    (trace_min 0.2)
-    (via_size 0.8)
-    (via_drill 0.4)
-    (via_min_size 0.4)
-    (via_min_drill 0.3)
-    (uvia_size 0.3)
-    (uvia_drill 0.1)
-    (uvias_allowed no)
-    (uvia_min_size 0.2)
-    (uvia_min_drill 0.1)
-    (edge_width 0.05)
-    (segment_width 0.2)
-    (pcb_text_width 0.3)
-    (pcb_text_size 1.5 1.5)
-    (mod_edge_width 0.12)
-    (mod_text_size 1 1)
-    (mod_text_width 0.15)
-    (pad_size 1.524 1.524)
-    (pad_drill 0.762)
     (pad_to_mask_clearance 0)
-    (aux_axis_origin 0 0)
-    (visible_elements FFFFFF7F)
     (pcbplotparams
-      (layerselection 0x010fc_ffffffff)
+      (layerselection 0x00010fc_ffffffff)
+      (disableapertmacros false)
       (usegerberextensions false)
       (usegerberattributes true)
       (usegerberadvancedattributes true)
       (creategerberjobfile false)
+      (svguseinch false)
+      (svgprecision 6)
       (excludeedgelayer true)
-      (linewidth 0.100000)
       (plotframeref false)
       (viasonmask false)
@@
       (hpglpenspeed 20)
       (hpglpendiameter 15.000000)
+      (dxfpolygonmode true)
+      (dxfimperialunits true)
+      (dxfusepcbnewfont true)
       (psnegative false)
       (psa4output false)
@@
       (plotvalue true)
       (plotinvisibletext false)
-      (padsonsilk false)
+      (sketchpadsonfab false)
       (subtractmaskfromsilk false)
       (outputformat 1)
@@
       (drillshape 0)
       (scaleselection 1)
-      (outputdirectory "../Fabrication/Spacer/"))
+      (outputdirectory "../Fabrication/Spacer/")
+    )
   )
   (net 0 "")
-  (net_class Default "This is the default net class."
-    (clearance 0.2)
-    (trace_width 0.25)
-    (via_dia 0.8)
-    (via_drill 0.4)
-    (uvia_dia 0.3)
-    (uvia_drill 0.1)
-  )
-  (gr_circle (center 175 100) (end 179 100) (layer B.SilkS) (width 0.12))
-  (gr_circle (center 120 100) (end 124 100) (layer B.SilkS) (width 0.12))
-  (gr_arc (start 176 101) (end 176 105) (angle -90) (layer Edge.Cuts) (width 0.05))
-  (gr_arc (start 176 99) (end 180 99) (angle -90) (layer Edge.Cuts) (width 0.05))
-  (gr_arc (start 119 101) (end 115 101) (angle -90) (layer Edge.Cuts) (width 0.05))
-  (gr_arc (start 119 99) (end 119 95) (angle -90) (layer Edge.Cuts) (width 0.05))
-  (gr_circle (center 175 100) (end 179 100) (layer F.SilkS) (width 0.12))
-  (gr_circle (center 175 100) (end 176.5 100) (layer Edge.Cuts) (width 0.05))
-  (gr_circle (center 120 100) (end 124 100) (layer F.SilkS) (width 0.12))
-  (gr_circle (center 120 100) (end 121.5 100) (layer Edge.Cuts) (width 0.05))
-  (gr_line (start 176 95) (end 119 95) (layer Edge.Cuts) (width 0.05))
-  (gr_line (start 180 101) (end 180 99) (layer Edge.Cuts) (width 0.05))
-  (gr_line (start 119 105) (end 176 105) (layer Edge.Cuts) (width 0.05))
-  (gr_line (start 115 99) (end 115 101) (layer Edge.Cuts) (width 0.05))
+  (gr_circle (center 175 100) (end 179 100) (layer "B.SilkS") (width 0.12) (fill none))
+  (gr_circle (center 120 100) (end 124 100) (layer "B.SilkS") (width 0.12) (fill none))
+  (gr_circle (center 175 100) (end 179 100) (layer "F.SilkS") (width 0.12) (fill none))
+  (gr_circle (center 120 100) (end 124 100) (layer "F.SilkS") (width 0.12) (fill none))
+  (gr_line (start 176 95) (end 119 95) (layer "Edge.Cuts") (width 0.05))
+  (gr_circle (center 175 100) (end 176.5 100) (layer "Edge.Cuts") (width 0.05) (fill none))
+  (gr_line (start 119 105) (end 176 105) (layer "Edge.Cuts") (width 0.05))
+  (gr_arc (start 119 105) (mid 116.171573 103.828427) (end 115 101) (layer "Edge.Cuts") (width 0.05))
+  (gr_arc (start 176 95) (mid 178.828427 96.171573) (end 180 99) (layer "Edge.Cuts") (width 0.05))
+  (gr_circle (center 120 100) (end 121.5 100) (layer "Edge.Cuts") (width 0.05) (fill none))
+  (gr_arc (start 180 101) (mid 178.828427 103.828427) (end 176 105) (layer "Edge.Cuts") (width 0.05))
+  (gr_arc (start 115 99) (mid 116.171573 96.171573) (end 119 95) (layer "Edge.Cuts") (width 0.05))
+  (gr_line (start 180 101) (end 180 99) (layer "Edge.Cuts") (width 0.05))
+  (gr_line (start 115 99) (end 115 101) (layer "Edge.Cuts") (width 0.05))
 )
